Commit message: Fix: Remove pi redefinition (xacro has built-in pi constant)

File: urdf/agribot.xacro (robot description, xacro)
@@ -1,6 +1,4 @@
 <?xml version="1.0"?>
 <robot name="agribot" xmlns:xacro="http://www.ros.org/wiki/xacro">
-  <!-- Constants -->
-  <xacro:property name="pi" value="3.1415926535897931"/>
   <!-- Materials -->
   <material name="grey"><color rgba="0.5 0.5 0.5 1.0"/></material>

Commit message: CRITICAL FIX: Correct dimensions from mm to meters (81cm wheelbase, 87cm track)

File: urdf/agribot.xacro (robot description, xacro)
@@ -26,19 +26,20 @@
   </link>
   <!-- V-Leg Macro: Creates leg and wheel assembly -->
+  <!-- Corrected dimensions: 81cm (0.81m) wheelbase, 87cm (0.87m) track -->
   <xacro:macro name="v_leg" params="prefix x_reflect y_reflect">
     <!-- Leg Link -->
     <link name="${prefix}_leg">
       <visual>
-        <origin xyz="${x_reflect*0.04} ${y_reflect*0.043} 0.32" rpy="0 0.5 0"/>
-        <geometry><box size="0.04 0.04 0.3"/></geometry>
+        <origin xyz="${x_reflect*0.2} ${y_reflect*0.2} 0.32" rpy="0 0.5 0"/>
+        <geometry><box size="0.05 0.05 0.4"/></geometry>
         <material name="grey"/>
       </visual>
       <collision>
-        <origin xyz="${x_reflect*0.04} ${y_reflect*0.043} 0.32" rpy="0 0.5 0"/>
-        <geometry><box size="0.04 0.04 0.3"/></geometry>
+        <origin xyz="${x_reflect*0.2} ${y_reflect*0.2} 0.32" rpy="0 0.5 0"/>
+        <geometry><box size="0.05 0.05 0.4"/></geometry>
       </collision>
       <inertial>
         <mass value="2.0"/>
-        <origin xyz="${x_reflect*0.04} ${y_reflect*0.043} 0.32"/>
+        <origin xyz="${x_reflect*0.2} ${y_reflect*0.2} 0.32"/>
         <inertia ixx="0.01" ixy="0" ixz="0" iyy="0.01" iyz="0" izz="0.01"/>
       </inertial>
@@ -65,8 +66,9 @@
     </link>
     <!-- Continuous joint for wheel rotation -->
+    <!-- Wheel positions: 0.405m (half of 0.81m wheelbase), 0.435m (half of 0.87m track) -->
     <joint name="${prefix}_wheel_joint" type="continuous">
       <parent link="${prefix}_leg"/>
       <child link="${prefix}_wheel"/>
-      <origin xyz="${x_reflect*0.0405} ${y_reflect*0.0435} 0.2025" rpy="${pi/2} 0 0"/>
+      <origin xyz="${x_reflect*0.405} ${y_reflect*0.435} 0.2025" rpy="${pi/2} 0 0"/>
       <axis xyz="0 0 1"/>
       <limit effort="300" velocity="10.0"/>
@@ -94,5 +96,5 @@
       <left_joint>front_left_wheel_joint</left_joint>
       <right_joint>front_right_wheel_joint</right_joint>
-      <wheel_separation>0.087</wheel_separation>
+      <wheel_separation>0.87</wheel_separation>
       <wheel_diameter>0.405</wheel_diameter>
       <max_wheel_torque>300</max_wheel_torque>

Commit message: Fix: Enlarge chassis and correct leg positioning for proper proportions

File: urdf/agribot.xacro (robot description, xacro)
@@ -5,70 +5,72 @@
   <material name="black"><color rgba="0.1 0.1 0.1 1.0"/></material>
   <!-- Base Link: High-clearance chassis at 450mm -->
+  <!-- Enlarged to 0.8m x 0.5m to match substantial steel frame in photo -->
   <link name="base_link">
     <visual>
       <origin xyz="0 0 0.45" rpy="0 0 0"/>
       <geometry>
-        <box size="0.2 0.2 0.05"/>
+        <box size="0.8 0.5 0.1"/>
       </geometry>
       <material name="grey"/>
     </visual>
     <collision>
-      <origin xyz="0 0 0.45"/>
+      <origin xyz="0 0 0.45" rpy="0 0 0"/>
       <geometry>
-        <box size="0.2 0.2 0.05"/>
+        <box size="0.8 0.5 0.1"/>
       </geometry>
     </collision>
     <inertial>
-      <mass value="40.0"/>
-      <origin xyz="0 0 0.45"/>
-      <inertia ixx="0.5" ixy="0" ixz="0" iyy="0.5" iyz="0" izz="0.5"/>
+      <mass value="50.0"/>
+      <origin xyz="0 0 0.45" rpy="0 0 0"/>
+      <inertia ixx="1.2" ixy="0" ixz="0" iyy="1.2" iyz="0" izz="1.2"/>
     </inertial>
   </link>
   <!-- V-Leg Macro: Creates leg and wheel assembly -->
   <!-- Corrected dimensions: 81cm (0.81m) wheelbase, 87cm (0.87m) track -->
+  <!-- Legs positioned at corners of chassis with proper flare for wide track -->
   <xacro:macro name="v_leg" params="prefix x_reflect y_reflect">
-    <!-- Leg Link -->
+    <!-- Leg Link: Thick square tubing (60mm) angled to reach wheels -->
     <link name="${prefix}_leg">
       <visual>
-        <origin xyz="${x_reflect*0.2} ${y_reflect*0.2} 0.32" rpy="0 0.5 0"/>
-        <geometry><box size="0.05 0.05 0.4"/></geometry>
+        <origin xyz="0 0 0.1" rpy="0 ${x_reflect * 0.4} 0"/>
+        <geometry><box size="0.06 0.06 0.4"/></geometry>
         <material name="grey"/>
       </visual>
       <collision>
-        <origin xyz="${x_reflect*0.2} ${y_reflect*0.2} 0.32" rpy="0 0.5 0"/>
-        <geometry><box size="0.05 0.05 0.4"/></geometry>
+        <origin xyz="0 0 0.1" rpy="0 ${x_reflect * 0.4} 0"/>
+        <geometry><box size="0.06 0.06 0.4"/></geometry>
       </collision>
       <inertial>
-        <mass value="2.0"/>
-        <origin xyz="${x_reflect*0.2} ${y_reflect*0.2} 0.32"/>
-        <inertia ixx="0.01" ixy="0" ixz="0" iyy="0.01" iyz="0" izz="0.01"/>
+        <mass value="2.5"/>
+        <origin xyz="0 0 0.1"/>
+        <inertia ixx="0.015" ixy="0" ixz="0" iyy="0.015" iyz="0" izz="0.015"/>
       </inertial>
     </link>
-    <!-- Fixed joint connecting leg to base -->
+    <!-- Fixed joint connecting leg to base at chassis corners -->
     <joint name="${prefix}_leg_joint" type="fixed">
       <parent link="base_link"/>
       <child link="${prefix}_leg"/>
-      <origin xyz="0 0 0"/>
+      <origin xyz="${x_reflect*0.4} ${y_reflect*0.25} 0.45" rpy="0 0 0"/>
     </joint>
     <!-- Wheel Link: 4.00-8 tire (405mm diameter, 0.2025m radius) -->
     <link name="${prefix}_wheel">
       <visual>
-        <geometry><cylinder radius="0.2025" length="0.101"/></geometry>
+        <geometry><cylinder radius="0.2025" length="0.12"/></geometry>
         <material name="black"/>
       </visual>
       <collision>
-        <geometry><cylinder radius="0.2025" length="0.101"/></geometry>
+        <geometry><cylinder radius="0.2025" length="0.12"/></geometry>
       </collision>
       <inertial>
-        <mass value="5.0"/>
-        <inertia ixx="0.06" ixy="0" ixz="0" iyy="0.06" iyz="0" izz="0.1"/>
+        <mass value="6.0"/>
+        <inertia ixx="0.07" ixy="0" ixz="0" iyy="0.07" iyz="0" izz="0.12"/>
       </inertial>
     </link>
     <!-- Continuous joint for wheel rotation -->
-    <!-- Wheel positions: 0.405m (half of 0.81m wheelbase), 0.435m (half of 0.87m track) -->
+    <!-- Wheel positions create 0.87m track width (0.25 chassis + 0.185 flare = 0.435m per side) -->
     <joint name="${prefix}_wheel_joint" type="continuous">
       <parent link="${prefix}_leg"/>
       <child link="${prefix}_wheel"/>
-      <origin xyz="${x_reflect*0.405} ${y_reflect*0.435} 0.2025" rpy="${pi/2} 0 0"/>
+      <origin xyz="${x_reflect*0.05} ${y_reflect*0.185} -0.2475" rpy="${-pi/2} 0 0"/>
       <axis xyz="0 0 1"/>
       <limit effort="300" velocity="10.0"/>

Commit message: Industrial scale fix: Enlarge chassis to 0.9m x 0.6m and adjust leg-to-wheel connections

File: urdf/agribot.xacro (robot description, xacro)
@@ -5,10 +5,10 @@
   <material name="black"><color rgba="0.1 0.1 0.1 1.0"/></material>
   <!-- Base Link: High-clearance chassis at 450mm -->
-  <!-- Enlarged to 0.8m x 0.5m to match substantial steel frame in photo -->
+  <!-- Industrial scale: 0.9m x 0.6m heavy steel frame that fills space between wheels -->
   <link name="base_link">
     <visual>
       <origin xyz="0 0 0.45" rpy="0 0 0"/>
       <geometry>
-        <box size="0.8 0.5 0.1"/>
+        <box size="0.9 0.6 0.08"/>
       </geometry>
       <material name="grey"/>
@@ -17,32 +17,32 @@
       <origin xyz="0 0 0.45" rpy="0 0 0"/>
       <geometry>
-        <box size="0.8 0.5 0.1"/>
+        <box size="0.9 0.6 0.08"/>
       </geometry>
     </collision>
     <inertial>
-      <mass value="50.0"/>
+      <mass value="60.0"/>
       <origin xyz="0 0 0.45" rpy="0 0 0"/>
-      <inertia ixx="1.2" ixy="0" ixz="0" iyy="1.2" iyz="0" izz="1.2"/>
+      <inertia ixx="1.5" ixy="0" ixz="0" iyy="2.0" iyz="0" izz="2.0"/>
     </inertial>
   </link>
   <!-- V-Leg Macro: Creates leg and wheel assembly -->
+  <!-- Industrial scale: Heavy frame with V-legs that extend to wheels -->
   <!-- Corrected dimensions: 81cm (0.81m) wheelbase, 87cm (0.87m) track -->
-  <!-- Legs positioned at corners of chassis with proper flare for wide track -->
   <xacro:macro name="v_leg" params="prefix x_reflect y_reflect">
-    <!-- Leg Link: Thick square tubing (60mm) angled to reach wheels -->
+    <!-- Leg Link: Thick square tubing (60mm) with sharper V-angle -->
     <link name="${prefix}_leg">
       <visual>
-        <origin xyz="0 0 0.1" rpy="0 ${x_reflect * 0.4} 0"/>
-        <geometry><box size="0.06 0.06 0.4"/></geometry>
+        <origin xyz="0 0 -0.12" rpy="0 ${x_reflect * 0.5} 0"/>
+        <geometry><box size="0.06 0.06 0.35"/></geometry>
         <material name="grey"/>
       </visual>
       <collision>
-        <origin xyz="0 0 0.1" rpy="0 ${x_reflect * 0.4} 0"/>
-        <geometry><box size="0.06 0.06 0.4"/></geometry>
+        <origin xyz="0 0 -0.12" rpy="0 ${x_reflect * 0.5} 0"/>
+        <geometry><box size="0.06 0.06 0.35"/></geometry>
       </collision>
       <inertial>
-        <mass value="2.5"/>
-        <origin xyz="0 0 0.1"/>
-        <inertia ixx="0.015" ixy="0" ixz="0" iyy="0.015" iyz="0" izz="0.015"/>
+        <mass value="3.0"/>
+        <origin xyz="0 0 -0.12"/>
+        <inertia ixx="0.02" ixy="0" ixz="0" iyy="0.02" iyz="0" izz="0.02"/>
       </inertial>
     </link>
@@ -51,5 +51,5 @@
       <parent link="base_link"/>
       <child link="${prefix}_leg"/>
-      <origin xyz="${x_reflect*0.4} ${y_reflect*0.25} 0.45" rpy="0 0 0"/>
+      <origin xyz="${x_reflect*0.4} ${y_reflect*0.3} 0.45" rpy="0 0 0"/>
     </joint>
     <!-- Wheel Link: 4.00-8 tire (405mm diameter, 0.2025m radius) -->
@@ -63,14 +63,14 @@
       </collision>
       <inertial>
-        <mass value="6.0"/>
-        <inertia ixx="0.07" ixy="0" ixz="0" iyy="0.07" iyz="0" izz="0.12"/>
+        <mass value="8.0"/>
+        <inertia ixx="0.1" ixy="0" ixz="0" iyy="0.1" iyz="0" izz="0.15"/>
       </inertial>
     </link>
     <!-- Continuous joint for wheel rotation -->
-    <!-- Wheel positions create 0.87m track width (0.25 chassis + 0.185 flare = 0.435m per side) -->
+    <!-- Wheel offset: 0.3m leg attachment + 0.135m wheel offset = 0.435m (half of 0.87m track) -->
     <joint name="${prefix}_wheel_joint" type="continuous">
       <parent link="${prefix}_leg"/>
       <child link="${prefix}_wheel"/>
-      <origin xyz="${x_reflect*0.05} ${y_reflect*0.185} -0.2475" rpy="${-pi/2} 0 0"/>
+      <origin xyz="${x_reflect*0.08} ${y_reflect*0.135} -0.2475" rpy="${-pi/2} 0 0"/>
       <axis xyz="0 0 1"/>
       <limit effort="300" velocity="10.0"/>

Commit message: High-clearance update: Raise chassis to 0.6m, adjust tip-over test, reduce soft-start rates

File: urdf/agribot.xacro (robot description, xacro)
@@ -4,45 +4,46 @@
   <material name="grey"><color rgba="0.5 0.5 0.5 1.0"/></material>
   <material name="black"><color rgba="0.1 0.1 0.1 1.0"/></material>
-  <!-- Base Link: High-clearance chassis at 450mm -->
-  <!-- Industrial scale: 0.9m x 0.6m heavy steel frame that fills space between wheels -->
+  <!-- Base Link: High-clearance chassis at 600mm -->
+  <!-- High-clearance agricultural design: 1.0m x 0.5m frame at 0.6m height -->
+  <!-- This creates significant clearance above 405mm tires, matching workshop photo -->
   <link name="base_link">
     <visual>
-      <origin xyz="0 0 0.45" rpy="0 0 0"/>
+      <origin xyz="0 0 0.6" rpy="0 0 0"/>
       <geometry>
-        <box size="0.9 0.6 0.08"/>
+        <box size="1.0 0.5 0.04"/>
       </geometry>
       <material name="grey"/>
     </visual>
     <collision>
-      <origin xyz="0 0 0.45" rpy="0 0 0"/>
+      <origin xyz="0 0 0.6" rpy="0 0 0"/>
       <geometry>
-        <box size="0.9 0.6 0.08"/>
+        <box size="1.0 0.5 0.04"/>
       </geometry>
     </collision>
     <inertial>
-      <mass value="60.0"/>
-      <origin xyz="0 0 0.45" rpy="0 0 0"/>
-      <inertia ixx="1.5" ixy="0" ixz="0" iyy="2.0" iyz="0" izz="2.0"/>
+      <mass value="70.0"/>
+      <origin xyz="0 0 0.6" rpy="0 0 0"/>
+      <inertia ixx="2.0" ixy="0" ixz="0" iyy="3.0" iyz="0" izz="3.0"/>
     </inertial>
   </link>
   <!-- V-Leg Macro: Creates leg and wheel assembly -->
-  <!-- Industrial scale: Heavy frame with V-legs that extend to wheels -->
+  <!-- High-clearance: Longer, more vertical legs to reach 0.6m chassis height -->
   <!-- Corrected dimensions: 81cm (0.81m) wheelbase, 87cm (0.87m) track -->
   <xacro:macro name="v_leg" params="prefix x_reflect y_reflect">
-    <!-- Leg Link: Thick square tubing (60mm) with sharper V-angle -->
+    <!-- Leg Link: Longer legs (0.55m) with more vertical angle for high clearance -->
     <link name="${prefix}_leg">
       <visual>
-        <origin xyz="0 0 -0.12" rpy="0 ${x_reflect * 0.5} 0"/>
-        <geometry><box size="0.06 0.06 0.35"/></geometry>
+        <origin xyz="0 0 -0.2" rpy="0 ${x_reflect * 0.3} 0"/>
+        <geometry><box size="0.05 0.05 0.55"/></geometry>
         <material name="grey"/>
       </visual>
       <collision>
-        <origin xyz="0 0 -0.12" rpy="0 ${x_reflect * 0.5} 0"/>
-        <geometry><box size="0.06 0.06 0.35"/></geometry>
+        <origin xyz="0 0 -0.2" rpy="0 ${x_reflect * 0.3} 0"/>
+        <geometry><box size="0.05 0.05 0.55"/></geometry>
       </collision>
       <inertial>
-        <mass value="3.0"/>
-        <origin xyz="0 0 -0.12"/>
-        <inertia ixx="0.02" ixy="0" ixz="0" iyy="0.02" iyz="0" izz="0.02"/>
+        <mass value="3.5"/>
+        <origin xyz="0 0 -0.2"/>
+        <inertia ixx="0.025" ixy="0" ixz="0" iyy="0.025" iyz="0" izz="0.025"/>
       </inertial>
     </link>
@@ -51,5 +52,5 @@
       <parent link="base_link"/>
       <child link="${prefix}_leg"/>
-      <origin xyz="${x_reflect*0.4} ${y_reflect*0.3} 0.45" rpy="0 0 0"/>
+      <origin xyz="${x_reflect*0.45} ${y_reflect*0.25} 0.6" rpy="0 0 0"/>
     </joint>
     <!-- Wheel Link: 4.00-8 tire (405mm diameter, 0.2025m radius) -->
@@ -68,9 +69,10 @@
     </link>
     <!-- Continuous joint for wheel rotation -->
-    <!-- Wheel offset: 0.3m leg attachment + 0.135m wheel offset = 0.435m (half of 0.87m track) -->
+    <!-- Wheel offset: 0.25m leg attachment + 0.185m wheel offset = 0.435m (half of 0.87m track) -->
+    <!-- Z offset: -0.3975m to place wheel at ground level (0.6m chassis - 0.2025m radius - 0.3975m = 0.0m) -->
     <joint name="${prefix}_wheel_joint" type="continuous">
       <parent link="${prefix}_leg"/>
       <child link="${prefix}_wheel"/>
-      <origin xyz="${x_reflect*0.08} ${y_reflect*0.135} -0.2475" rpy="${-pi/2} 0 0"/>
+      <origin xyz="${x_reflect*0.06} ${y_reflect*0.185} -0.3975" rpy="${-pi/2} 0 0"/>
       <axis xyz="0 0 1"/>
       <limit effort="300" velocity="10.0"/>

Commit message: Update for 22.5:1 total reduction (10:1 gearbox + 2.25:1 chain) - add gearbox friction, torque monitoring, and controller gains

File: urdf/agribot.xacro (robot description, xacro)
@@ -71,4 +71,5 @@
     <!-- Wheel offset: 0.25m leg attachment + 0.185m wheel offset = 0.435m (half of 0.87m track) -->
     <!-- Z offset: -0.3975m to place wheel at ground level (0.6m chassis - 0.2025m radius - 0.3975m = 0.0m) -->
+    <!-- Total reduction: 22.5:1 (10:1 gearbox + 2.25:1 chain) -->
     <joint name="${prefix}_wheel_joint" type="continuous">
       <parent link="${prefix}_leg"/>
@@ -76,7 +77,12 @@
       <origin xyz="${x_reflect*0.06} ${y_reflect*0.185} -0.3975" rpy="${-pi/2} 0 0"/>
       <axis xyz="0 0 1"/>
+      <!-- Max effort accounts for 22.5:1 reduction: 300Nm * 22.5 = 6750Nm at wheel -->
+      <!-- But we cap at 300Nm to match gearbox rating -->
       <limit effort="300" velocity="10.0"/>
+      <!-- Gearbox friction and damping (10:1 gearbox has internal resistance) -->
+      <dynamics damping="50.0" friction="10.0"/>
     </joint>
     <!-- Gazebo friction parameters for skid-steer -->
+    <!-- Gearbox friction acts as natural brake when power is cut -->
     <gazebo reference="${prefix}_wheel">
       <mu1>1.1</mu1>
@@ -84,4 +90,14 @@
       <kp>1000000.0</kp>
       <kd>10.0</kd>
+      <!-- Gearbox damping to simulate 10:1 gearbox internal resistance -->
+      <minDepth>0.001</minDepth>
+      <maxVel>1.0</maxVel>
+    </gazebo>
+    <!-- Gearbox joint damping (simulates 10:1 gearbox backlash and friction) -->
+    <gazebo reference="${prefix}_wheel_joint">
+      <implicitSpringDamper>true</implicitSpringDamper>
+      <stopCfm>0.1</stopCfm>
+      <stopErp>0.2</stopErp>
+      <fudgeFactor>0.5</fudgeFactor>
     </gazebo>
   </xacro:macro>

Commit message: Add jackshaft model, dual-chain damping, and belly clearance test for 40cm crops

File: urdf/agribot.xacro (robot description, xacro)
@@ -68,18 +68,50 @@
       </inertial>
     </link>
+    <!-- Jackshaft Link: 36T sprocket on middle jackshaft (two-stage chain drive) -->
+    <!-- 16T (Gearbox) → 36T (Jackshaft) → 16T (Wheel) = 2.25:1 chain reduction -->
+    <link name="${prefix}_jackshaft">
+      <visual>
+        <origin xyz="0 0 0" rpy="0 0 0"/>
+        <geometry>
+          <cylinder radius="0.08" length="0.06"/>  <!-- 36T sprocket ~16cm diameter -->
+        </geometry>
+        <material name="grey"/>
+      </visual>
+      <collision>
+        <geometry>
+          <cylinder radius="0.08" length="0.06"/>
+        </geometry>
+      </collision>
+      <inertial>
+        <!-- Rotating mass of jackshaft + 36T sprocket acts as flywheel -->
+        <mass value="2.5"/>  <!-- Jackshaft + large sprocket weight -->
+        <inertia ixx="0.02" ixy="0" ixz="0" iyy="0.02" iyz="0" izz="0.02"/>
+      </inertial>
+    </link>
+    <!-- Jackshaft joint: Connects to leg at middle height (preserves 0.6m clearance) -->
+    <joint name="${prefix}_jackshaft_joint" type="continuous">
+      <parent link="${prefix}_leg"/>
+      <child link="${prefix}_jackshaft"/>
+      <!-- Positioned in middle of leg to keep 36T sprocket protected and high -->
+      <origin xyz="${x_reflect*0.02} ${y_reflect*0.1} -0.15" rpy="${pi/2} 0 0"/>
+      <axis xyz="0 0 1"/>
+      <limit effort="300" velocity="10.0"/>
+      <!-- Dual-chain damping: two chains = more backlash and damping -->
+      <dynamics damping="75.0" friction="15.0"/>
+    </joint>
     <!-- Continuous joint for wheel rotation -->
     <!-- Wheel offset: 0.25m leg attachment + 0.185m wheel offset = 0.435m (half of 0.87m track) -->
     <!-- Z offset: -0.3975m to place wheel at ground level (0.6m chassis - 0.2025m radius - 0.3975m = 0.0m) -->
-    <!-- Total reduction: 22.5:1 (10:1 gearbox + 2.25:1 chain) -->
+    <!-- Total reduction: 22.5:1 (10:1 gearbox + 2.25:1 chain: 16T→36T=2.25:1, 16T→16T=1:1) -->
     <joint name="${prefix}_wheel_joint" type="continuous">
-      <parent link="${prefix}_leg"/>
+      <parent link="${prefix}_jackshaft"/>  <!-- Wheel driven from jackshaft, not directly from leg -->
       <child link="${prefix}_wheel"/>
-      <origin xyz="${x_reflect*0.06} ${y_reflect*0.185} -0.3975" rpy="${-pi/2} 0 0"/>
+      <origin xyz="${x_reflect*0.04} ${y_reflect*0.085} -0.2475" rpy="${-pi/2} 0 0"/>
       <axis xyz="0 0 1"/>
       <!-- Max effort accounts for 22.5:1 reduction: 300Nm * 22.5 = 6750Nm at wheel -->
       <!-- But we cap at 300Nm to match gearbox rating -->
       <limit effort="300" velocity="10.0"/>
-      <!-- Gearbox friction and damping (10:1 gearbox has internal resistance) -->
-      <dynamics damping="50.0" friction="10.0"/>
+      <!-- Second chain stage: 16T to 16T (1:1) - less damping than first stage -->
+      <dynamics damping="25.0" friction="5.0"/>
     </joint>
     <!-- Gazebo friction parameters for skid-steer -->

Commit message: Fix: Keep wheel attached to leg, jackshaft as separate rotating element for inertia

File: urdf/agribot.xacro (robot description, xacro)
@@ -70,4 +70,5 @@
     <!-- Jackshaft Link: 36T sprocket on middle jackshaft (two-stage chain drive) -->
     <!-- 16T (Gearbox) → 36T (Jackshaft) → 16T (Wheel) = 2.25:1 chain reduction -->
+    <!-- Jackshaft positioned in middle of leg to preserve 0.6m ground clearance -->
     <link name="${prefix}_jackshaft">
       <visual>
@@ -85,17 +86,18 @@
       <inertial>
         <!-- Rotating mass of jackshaft + 36T sprocket acts as flywheel -->
+        <!-- Adds rotational inertia - robot won't stop instantly when motor stops -->
         <mass value="2.5"/>  <!-- Jackshaft + large sprocket weight -->
         <inertia ixx="0.02" ixy="0" ixz="0" iyy="0.02" iyz="0" izz="0.02"/>
       </inertial>
     </link>
-    <!-- Jackshaft joint: Connects to leg at middle height (preserves 0.6m clearance) -->
+    <!-- Jackshaft joint: Rotating element in middle of leg (simulates 16T→36T chain stage) -->
     <joint name="${prefix}_jackshaft_joint" type="continuous">
       <parent link="${prefix}_leg"/>
       <child link="${prefix}_jackshaft"/>
-      <!-- Positioned in middle of leg to keep 36T sprocket protected and high -->
+      <!-- Positioned in middle of leg to keep 36T sprocket protected and high (preserves clearance) -->
       <origin xyz="${x_reflect*0.02} ${y_reflect*0.1} -0.15" rpy="${pi/2} 0 0"/>
       <axis xyz="0 0 1"/>
       <limit effort="300" velocity="10.0"/>
-      <!-- Dual-chain damping: two chains = more backlash and damping -->
+      <!-- First chain stage damping: 16T→36T (2.25:1) - higher damping from larger sprocket -->
       <dynamics damping="75.0" friction="15.0"/>
     </joint>
@@ -104,14 +106,16 @@
     <!-- Z offset: -0.3975m to place wheel at ground level (0.6m chassis - 0.2025m radius - 0.3975m = 0.0m) -->
     <!-- Total reduction: 22.5:1 (10:1 gearbox + 2.25:1 chain: 16T→36T=2.25:1, 16T→16T=1:1) -->
+    <!-- Note: Wheel is directly attached to leg for proper ground contact, but driven via chain from jackshaft -->
     <joint name="${prefix}_wheel_joint" type="continuous">
-      <parent link="${prefix}_jackshaft"/>  <!-- Wheel driven from jackshaft, not directly from leg -->
+      <parent link="${prefix}_leg"/>  <!-- Wheel attached to leg for ground contact -->
       <child link="${prefix}_wheel"/>
-      <origin xyz="${x_reflect*0.04} ${y_reflect*0.085} -0.2475" rpy="${-pi/2} 0 0"/>
+      <origin xyz="${x_reflect*0.06} ${y_reflect*0.185} -0.3975" rpy="${-pi/2} 0 0"/>
       <axis xyz="0 0 1"/>
       <!-- Max effort accounts for 22.5:1 reduction: 300Nm * 22.5 = 6750Nm at wheel -->
       <!-- But we cap at 300Nm to match gearbox rating -->
       <limit effort="300" velocity="10.0"/>
-      <!-- Second chain stage: 16T to 16T (1:1) - less damping than first stage -->
-      <dynamics damping="25.0" friction="5.0"/>
+      <!-- Second chain stage: 16T to 16T (1:1) - includes jackshaft flywheel inertia effect -->
+      <!-- Dual-chain system: increased backlash and damping from two chains -->
+      <dynamics damping="50.0" friction="10.0"/>
     </joint>
     <!-- Gazebo friction parameters for skid-steer -->
