Commit message: Add basic teleop test for Step 34 jump verification with 75kg mass and proper chain damping

File: urdf/agribot.xacro (robot description, xacro)
@@ -99,6 +99,7 @@
       <axis xyz="0 0 1"/>
       <limit effort="300" velocity="10.0"/>
-      <!-- First chain stage damping: 16T→36T (2.25:1) - higher damping from larger sprocket -->
-      <dynamics damping="75.0" friction="15.0"/>
+      <!-- First chain stage damping: 16T→36T (2.25:1) - Royal Enfield chain resistance -->
+      <!-- High damping from 10:1 gearbox + dual-chain setup -->
+      <dynamics damping="2.5" friction="1.5"/>
     </joint>
     <!-- Continuous joint for wheel rotation -->
@@ -116,6 +117,6 @@
       <limit effort="300" velocity="10.0"/>
       <!-- Second chain stage: 16T to 16T (1:1) - includes jackshaft flywheel inertia effect -->
-      <!-- Dual-chain system: increased backlash and damping from two chains -->
-      <dynamics damping="50.0" friction="10.0"/>
+      <!-- Dual-chain system: Royal Enfield chain resistance with 22.5:1 total reduction -->
+      <dynamics damping="2.5" friction="1.5"/>
     </joint>
     <!-- Gazebo friction parameters for skid-steer -->

Commit message: Fix: Update base mass to 75kg and add teleop test instructions

File: urdf/agribot.xacro (robot description, xacro)
@@ -22,7 +22,8 @@
     </collision>
     <inertial>
-      <mass value="70.0"/>
+      <!-- Total mass: 75kg (base + wheels + jackshafts + chains) -->
+      <mass value="75.0"/>
       <origin xyz="0 0 0.6" rpy="0 0 0"/>
-      <inertia ixx="2.0" ixy="0" ixz="0" iyy="3.0" iyz="0" izz="3.0"/>
+      <inertia ixx="2.5" ixy="0" ixz="0" iyy="3.5" iyz="0" izz="3.5"/>
     </inertial>
   </link>
