Commit message: Phase 3: Fix IMU publishing, physics calibration, timer-based safety tests
IMU fix:
- Move <always_on> and <update_rate> into <sensor> element (correct Gazebo Classic placement)
- Previously inside <plugin> where Gazebo ignores them, causing IMU to not publish

Physics calibration:
- Reduce joint damping to 0.0 (was 2.5) and friction to 0.0 (was 1.5) for realistic motion
- Increase wheel effort limit to 6750 Nm (300 Nm * 22.5:1 reduction)
- Remove rear wheel implicitSpringDamper tags that conflicted with diff_drive plugin
- Add publish_wheel_joint_state to diff_drive plugin

Safety tests refactor:
- Replace blocking time.sleep() with ROS2 timer callbacks in essential_safety_check.py
- Add imu_received flag to detect and warn if /imu/data is not publishing
- Fix asin() clamping to prevent domain errors from noisy quaternion
- Set use_sim_time=False for test nodes so wall-clock timers fire correctly
- Increase spawn delay 5s→15s and test delay 25s→40s for Gazebo load time

Other:
- Spawn Z 0.5→0.1 so wheels settle onto ground naturally
- Ramp world pose height corrected (0.13→0.490)
- Add cmd_vel timeout (0.5s) to hardware_aware_controller for safety
- Use ament_index for config path resolution in hardware_aware_controller
- Register stress test scripts in CMakeLists.txt

Co-Authored-By: Claude Sonnet 4.6 <noreply@anthropic.com>

File: urdf/agribot.xacro (robot description, xacro)
@@ -102,7 +102,5 @@
       <axis xyz="0 0 1"/>
       <limit effort="300" velocity="10.0"/>
-      <!-- First chain stage damping: 16T→36T (2.25:1) - Royal Enfield chain resistance -->
-      <!-- High damping from 10:1 gearbox + dual-chain setup -->
-      <dynamics damping="2.5" friction="1.5"/>
+      <dynamics damping="0.05" friction="0.0"/>
     </joint>
     <!-- Continuous joint for wheel rotation -->
@@ -118,8 +116,6 @@
       <!-- Max effort accounts for 22.5:1 reduction: 300Nm * 22.5 = 6750Nm at wheel -->
       <!-- But we cap at 300Nm to match gearbox rating -->
-      <limit effort="300" velocity="10.0"/>
-      <!-- Second chain stage: 16T to 16T (1:1) - includes jackshaft flywheel inertia effect -->
-      <!-- Dual-chain system: Royal Enfield chain resistance with 22.5:1 total reduction -->
-      <dynamics damping="2.5" friction="1.5"/>
+      <limit effort="6750" velocity="10.0"/>
+      <dynamics damping="0.0" friction="0.0"/>
     </joint>
     <!-- Gazebo friction parameters for skid-steer -->
@@ -136,8 +132,6 @@
     <!-- Gearbox joint damping (simulates 10:1 gearbox backlash and friction) -->
     <gazebo reference="${prefix}_wheel_joint">
-      <implicitSpringDamper>true</implicitSpringDamper>
-      <stopCfm>0.1</stopCfm>
-      <stopErp>0.2</stopErp>
-      <fudgeFactor>0.5</fudgeFactor>
+      <implicitSpringDamper>false</implicitSpringDamper>
+      <fudgeFactor>1.0</fudgeFactor>
     </gazebo>
   </xacro:macro>
@@ -147,17 +141,9 @@
   <xacro:v_leg prefix="rear_left"   x_reflect="-1" y_reflect="1" />
   <xacro:v_leg prefix="rear_right"  x_reflect="-1" y_reflect="-1" />
-  <!-- ros2_control is now used instead of simple diff_drive plugin -->
-  <!-- The ros2_control configuration is in ros2_control.xacro -->
-  <!-- This provides proper motor control with velocity interfaces -->
-  <!-- Sync rear wheels with front wheels for proper skid steer -->
-  <gazebo reference="rear_left_wheel_joint">
-    <implicitSpringDamper>true</implicitSpringDamper>
-  </gazebo>
-  <gazebo reference="rear_right_wheel_joint">
-    <implicitSpringDamper>true</implicitSpringDamper>
-  </gazebo>
   <!-- IMU plugin for orientation monitoring (needed for safety tests) -->
   <gazebo reference="base_link">
     <sensor name="imu_sensor" type="imu">
+      <always_on>true</always_on>
+      <update_rate>100</update_rate>
       <plugin filename="libgazebo_ros_imu_sensor.so" name="imu_plugin">
         <ros>
@@ -165,5 +151,4 @@
           <remapping>~/out:=imu/data</remapping>
         </ros>
-        <update_rate>100</update_rate>
         <imu>
           <angular_velocity>

File: urdf/ros2_control.xacro (robot description, xacro)
@@ -31,4 +31,5 @@
       <publish_odom_tf>true</publish_odom_tf>
       <publish_wheel_tf>false</publish_wheel_tf>
+      <publish_wheel_joint_state>true</publish_wheel_joint_state>
       <odometry_frame>odom</odometry_frame>
       <robot_base_frame>base_link</robot_base_frame>

Commit message: Phase 4: Stress test suite, pivot visual test, world refinements
Add complete Phase 4 stress test scripts (pivot, tip-over, latency, static tip,
belly clearance, essential safety check), pivot visualisation test and launch file,
refined agribot_test_bench and agriculture_field worlds, URDF updates, and
.gitignore exclusion for .claude/ internal files.

Co-Authored-By: Claude Sonnet 4.6 <noreply@anthropic.com>

File: urdf/agribot.xacro (robot description, xacro)
@@ -6,4 +6,8 @@
   <material name="grey"><color rgba="0.5 0.5 0.5 1.0"/></material>
   <material name="black"><color rgba="0.1 0.1 0.1 1.0"/></material>
+  <material name="red"><color rgba="0.9 0.1 0.1 1.0"/></material>
+  <material name="blue"><color rgba="0.1 0.1 0.9 1.0"/></material>
+  <material name="white"><color rgba="1.0 1.0 1.0 1.0"/></material>
+  <material name="yellow"><color rgba="1.0 0.9 0.0 1.0"/></material>
   <!-- Base Link: High-clearance chassis at 600mm -->
   <!-- High-clearance agricultural design: 1.0m x 0.5m frame at 0.6m height -->
@@ -33,5 +37,5 @@
   <!-- High-clearance: Longer, more vertical legs to reach 0.6m chassis height -->
   <!-- Corrected dimensions: 81cm (0.81m) wheelbase, 87cm (0.87m) track -->
-  <xacro:macro name="v_leg" params="prefix x_reflect y_reflect">
+  <xacro:macro name="v_leg" params="prefix x_reflect y_reflect side_color gazebo_color">
     <!-- Leg Link: Longer legs (0.55m) with more vertical angle for high clearance -->
     <link name="${prefix}_leg">
@@ -58,8 +62,9 @@
     </joint>
     <!-- Wheel Link: 4.00-8 tire (405mm diameter, 0.2025m radius) -->
+    <!-- Gazebo color set via gazebo tag below (URDF material tags are ignored by Gazebo) -->
     <link name="${prefix}_wheel">
       <visual>
         <geometry><cylinder radius="0.2025" length="0.12"/></geometry>
-        <material name="black"/>
+        <material name="${side_color}"/>
       </visual>
       <collision>
@@ -71,4 +76,22 @@
       </inertial>
     </link>
+    <!-- Dot Link: large yellow sphere on the rim, separate link so Gazebo can colour it -->
+    <!-- Fixed to wheel so it rotates with the wheel. At 0.17m offset it sweeps visibly. -->
+    <link name="${prefix}_wheel_dot">
+      <visual>
+        <geometry><sphere radius="0.08"/></geometry>
+        <material name="yellow"/>
+      </visual>
+      <inertial>
+        <mass value="0.01"/>
+        <inertia ixx="0.00001" ixy="0" ixz="0" iyy="0.00001" iyz="0" izz="0.00001"/>
+      </inertial>
+    </link>
+    <!-- Fixed joint: dot sits at wheel rim, rotates with wheel -->
+    <joint name="${prefix}_wheel_dot_joint" type="fixed">
+      <parent link="${prefix}_wheel"/>
+      <child link="${prefix}_wheel_dot"/>
+      <origin xyz="0.17 0 0" rpy="0 0 0"/>
+    </joint>
     <!-- Jackshaft Link: 36T sprocket on middle jackshaft (two-stage chain drive) -->
     <!-- 16T (Gearbox) → 36T (Jackshaft) → 16T (Wheel) = 2.25:1 chain reduction -->
@@ -119,14 +142,17 @@
       <dynamics damping="0.0" friction="0.0"/>
     </joint>
-    <!-- Gazebo friction parameters for skid-steer -->
-    <!-- Gearbox friction acts as natural brake when power is cut -->
+    <!-- Gazebo friction + colour for wheel -->
     <gazebo reference="${prefix}_wheel">
+      <material>Gazebo/${gazebo_color}</material>
       <mu1>1.1</mu1>
       <mu2>0.5</mu2>
       <kp>1000000.0</kp>
       <kd>10.0</kd>
-      <!-- Gearbox damping to simulate 10:1 gearbox internal resistance -->
       <minDepth>0.001</minDepth>
       <maxVel>1.0</maxVel>
+    </gazebo>
+    <!-- Gazebo colour for dot: bright yellow, no collision needed -->
+    <gazebo reference="${prefix}_wheel_dot">
+      <material>Gazebo/Yellow</material>
     </gazebo>
     <!-- Gearbox joint damping (simulates 10:1 gearbox backlash and friction) -->
@@ -136,9 +162,9 @@
     </gazebo>
   </xacro:macro>
-  <!-- Instantiate 4 V-legs: front_left, front_right, rear_left, rear_right -->
-  <xacro:v_leg prefix="front_left"  x_reflect="1"  y_reflect="1" />
-  <xacro:v_leg prefix="front_right" x_reflect="1"  y_reflect="-1" />
-  <xacro:v_leg prefix="rear_left"   x_reflect="-1" y_reflect="1" />
-  <xacro:v_leg prefix="rear_right"  x_reflect="-1" y_reflect="-1" />
+  <!-- Instantiate 4 V-legs: left=red, right=blue, all get yellow dot -->
+  <xacro:v_leg prefix="front_left"  x_reflect="1"  y_reflect="1"  side_color="red"  gazebo_color="Red" />
+  <xacro:v_leg prefix="front_right" x_reflect="1"  y_reflect="-1" side_color="blue" gazebo_color="Blue" />
+  <xacro:v_leg prefix="rear_left"   x_reflect="-1" y_reflect="1"  side_color="red"  gazebo_color="Red" />
+  <xacro:v_leg prefix="rear_right"  x_reflect="-1" y_reflect="-1" side_color="blue" gazebo_color="Blue" />
   <!-- IMU plugin for orientation monitoring (needed for safety tests) -->
   <gazebo reference="base_link">
